File: kicad/mt_reflowcnt/mt_reflowcnt.kicad_pcb (KiCad board)
At the start: 2 copper layers, 150.9 x 53.3 mm, 44 parts, among them IC1 TXB0101DBVR, IC2 TXB0101DBVR, IC3 MAX31855KASA+, IC4 NUP2105LT1G, IC5 TXB0101DBVR, J1 Conn_01x04, J2 PCC-SMP, P1 Power, P2 Analog, P3 Digital, P4 Digital, P5 CONN_01X01, P6 CONN_01X01, P7 CONN_01X01, P8 CONN_01X01, U1 SC2004CS_B

Commit message: first refined version. add more thermocouple and add one more relay control.
Parts:
- added C10: 0.01u, Capacitor_SMD:C_0805_2012Metric_Pad1.18x1.45mm_HandSolder, F.Cu at (232.6, 97.2)
- added C9: 0.01u, Capacitor_SMD:C_0805_2012Metric_Pad1.18x1.45mm_HandSolder, F.Cu at (211.8, 97.2)
- added D3: LED_Small, LED_SMD:LED_0805_2012Metric_Pad1.15x1.40mm_HandSolder, F.Cu at (254.5, 105.7)
- added IC6: NUP2105LT1G, LibraryLoader:SOT96P237X111-3N, F.Cu at (190.5, 101.0)
- added IC7: NUP2105LT1G, LibraryLoader:SOT96P237X111-3N, F.Cu at (211.8, 101.0)
- added IC8: NUP2105LT1G, LibraryLoader:SOT96P237X111-3N, F.Cu at (232.5, 101.0)
- added J3: PCC-SMP, mt_reflowcnt:PCC-SMP, F.Cu at (211.6, 84.7)
- added J4: PCC-SMP, mt_reflowcnt:PCC-SMP, F.Cu at (232.5, 84.7)
- added J5: Conn_01x01, Connector_PinSocket_2.54mm:PinSocket_1x01_P2.54mm_Vertical, F.Cu at (114.0, 123.6)
- added J6: Conn_01x01, Connector_PinSocket_2.54mm:PinSocket_1x01_P2.54mm_Vertical, F.Cu at (114.3, 76.3)
- added J7: Conn_01x01, Connector_PinSocket_2.54mm:PinSocket_1x01_P2.54mm_Vertical, F.Cu at (256.3, 115.7)
- added J8: Conn_01x01, Connector_PinSocket_2.54mm:PinSocket_1x01_P2.54mm_Vertical, F.Cu at (254.5, 85.2)
- added L3: 470ohm, Inductor_SMD:L_0603_1608Metric_Pad1.05x0.95mm_HandSolder, F.Cu at (204.7, 96.3)
- added L4: 470ohm, Inductor_SMD:L_0603_1608Metric_Pad1.05x0.95mm_HandSolder, F.Cu at (218.4, 96.3)
- added L5: 470ohm, Inductor_SMD:L_0603_1608Metric_Pad1.05x0.95mm_HandSolder, F.Cu at (225.7, 96.3)
- added L6: 470ohm, Inductor_SMD:L_0603_1608Metric_Pad1.05x0.95mm_HandSolder, F.Cu at (239.4, 96.3)
- added R13: 10k, Resistor_SMD:R_0805_2012Metric_Pad1.20x1.40mm_HandSolder, F.Cu at (125.2, 82.2)
- added R14: DNP, Resistor_SMD:R_0805_2012Metric_Pad1.20x1.40mm_HandSolder, F.Cu at (149.6, 104.5)
- added R15: DNP, Resistor_SMD:R_0805_2012Metric_Pad1.20x1.40mm_HandSolder, F.Cu at (152.1, 103.3)
- added R16: DNP, Resistor_SMD:R_0805_2012Metric_Pad1.20x1.40mm_HandSolder, F.Cu at (154.6, 101.2)
- added R17: DNP, Resistor_SMD:R_0805_2012Metric_Pad1.20x1.40mm_HandSolder, F.Cu at (157.0, 99.7)
- added R18: DNP, Resistor_SMD:R_0805_2012Metric_Pad1.20x1.40mm_HandSolder, F.Cu at (172.5, 93.3)
- C5: value 0.01u -> 0.1u
- C8: value 0.1u -> 0.01u
- IC1: value TXB0101DBVR -> TXB0104D; footprint LibraryLoader:SOT95P280X145-6N -> LibraryLoader:SOIC127P600X175-14N
- IC4: value NUP2105LT1G -> MAX31855KASA+; footprint LibraryLoader:SOT96P237X111-3N -> LibraryLoader:SOIC127P600X175-8N
- IC5: value TXB0101DBVR -> MAX31855KASA+; footprint LibraryLoader:SOT95P280X145-6N -> LibraryLoader:SOIC127P600X175-8N
- J1: value Conn_01x04 -> Conn_01x06; footprint Connector_PinHeader_2.54mm:PinHeader_1x04_P2.54mm_Vertical -> Connector_PinHeader_2.54mm:PinHeader_1x06_P2.54mm_Vertical
- R11: value 10k -> 33
- R2: value N6L50T0C-203-3030 -> 220; footprint LibraryLoader:N6L50T0C2033030 -> Resistor_SMD:R_0805_2012Metric_Pad1.20x1.40mm_HandSolder
- R3: value 220 -> N6L50T0C-203-3030; footprint Resistor_SMD:R_0805_2012Metric_Pad1.20x1.40mm_HandSolder -> LibraryLoader:N6L50T0C2033030
- R5: value 33 -> 220
- moved R2 136.7 mm to (254.5, 93.0), turned to 180 degrees
- moved R5 116.1 mm to (254.5, 103.1)
- moved R3 92.7 mm to (116.8, 99.5), turned to 180 degrees
- moved IC5 67.4 mm to (232.4, 108.1), turned to -90 degrees
- moved C7 67.0 mm to (227.3, 105.3)
- moved D1 50.9 mm to (254.5, 95.5), turned to 180 degrees
- moved J1 50.1 mm to (258.8, 93.0), turned to 0 degrees
- moved D2 39.5 mm to (254.5, 100.6), turned to 180 degrees
- moved R4 35.6 mm to (254.5, 98.0), turned to 180 degrees
- moved R12 33.1 mm to (125.5, 114.7), turned to 90 degrees
- moved C8 24.4 mm to (190.5, 97.2), turned to 180 degrees
- moved IC4 22.8 mm to (211.8, 108.1)
- moved R11 22.0 mm to (130.6, 91.8)
- moved C6 21.8 mm to (206.8, 105.3)
- moved R7 21.7 mm to (130.6, 102.0), turned to 180 degrees
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Connections:
- C3 pad 1: +3V3 -> +3.3V
- C4 pad 1: +3V3 -> +3.3V
- C5 pad 1: Net-(C5-Pad1) -> +3.3V
- C5 pad 2: Net-(C5-Pad2) -> GND
- C6 pad 1: +3V3 -> +3.3V
- C7 pad 1: +5V -> +3.3V
- C8 pad 1: +3V3 -> Net-(C8-Pad1)
- C8 pad 2: GND -> Net-(C8-Pad2)
- IC1 pad 1: +5V -> +3.3V
- IC1 pad 2: GND -> Net-(IC1-Pad2)
- IC1 pad 3: /13(SCK) -> Net-(IC3-Pad6)
- IC1 pad 4: Net-(IC3-Pad5) -> Net-(IC1-Pad4)
- IC1 pad 5: +5V -> Net-(IC5-Pad6)
- IC1 pad 6: +3V3 -> unconnected-(IC1-Pad6)
- IC2 pad 1: +5V -> +3.3V
- IC2 pad 2: GND -> Net-(IC2-Pad2)
- IC2 pad 3: /10(**/SS) -> GND
- IC2 pad 4: Net-(IC3-Pad6) -> /12(MISO)
- IC2 pad 5: +5V -> +3.3V
- IC2 pad 6: +3V3 -> +5V
- IC3 pad 2: Net-(C5-Pad2) -> Net-(C8-Pad1)
- IC3 pad 3: Net-(C5-Pad1) -> Net-(C8-Pad2)
- IC3 pad 4: +3V3 -> +3.3V
- IC3 pad 5: Net-(IC3-Pad5) -> Net-(IC1-Pad2)
- IC3 pad 7: Net-(IC3-Pad7) -> Net-(IC2-Pad2)
- IC4 pad 1: Net-(C5-Pad2) -> GND
- IC4 pad 2: Net-(C5-Pad1) -> Net-(C9-Pad1)
- IC4 pad 3: GND -> Net-(C9-Pad2)
- IC5 pad 1: +5V -> GND
- IC5 pad 2: GND -> Net-(C10-Pad1)
- IC5 pad 3: /12(MISO) -> Net-(C10-Pad2)
- IC5 pad 4: Net-(IC3-Pad7) -> +3.3V
- IC5 pad 5: +5V -> Net-(IC1-Pad2)
- IC5 pad 6: +3V3 -> Net-(IC5-Pad6)
- J1 pad 3: GND -> /A1
- J1 pad 4: /A1 -> GND
- L1 pad 1: Net-(C5-Pad1) -> Net-(C8-Pad2)
- L2 pad 1: Net-(C5-Pad2) -> Net-(C8-Pad1)
- P1 pad 4: +3V3 -> +3.3V
- R10 pad 2: /7 -> /6(**)
- R11 pad 1: +5V -> Net-(R11-Pad1)
- R11 pad 2: /8 -> /7
- R12 pad 2: /Reset -> /8
- R2 pad 1: Net-(R1-Pad2) -> /A0
- R2 pad 2: GND -> Net-(D1-Pad2)
- R3 pad 1: /A0 -> Net-(R1-Pad2)
- R3 pad 2: Net-(D1-Pad2) -> GND
- R5 pad 1: Net-(R5-Pad1) -> /9(**)
- R5 pad 2: /2 -> Net-(D3-Pad2)
- R6 pad 2: /3(**) -> /2
- R7 pad 2: /4 -> /3(**)
- R8 pad 2: /5(**) -> /4
- R9 pad 2: /6(**) -> /5(**)
- U1 pad 11: Net-(R7-Pad1) -> Net-(R8-Pad1)
- U1 pad 12: Net-(R8-Pad1) -> Net-(R9-Pad1)
- U1 pad 13: Net-(R9-Pad1) -> Net-(R10-Pad1)
- U1 pad 14: Net-(R10-Pad1) -> Net-(R11-Pad1)
- U1 pad 3: Net-(R2-Pad3) -> Net-(R3-Pad3)
- U1 pad 4: Net-(R5-Pad1) -> Net-(R6-Pad1)
- U1 pad 6: Net-(R6-Pad1) -> Net-(R7-Pad1)
Routing:
- net GND: track 286.7 -> 652.3 mm, vias 16 -> 49
- net +3.3V: track 0.00 -> 147.4 mm, vias 0 -> 3
- net /9(**): track 0.00 -> 142.1 mm, vias 0 -> 2
- net +3V3: track 92.4 -> 0.00 mm, vias 3 -> 0
- net Net-(IC2-Pad2): track 0.00 -> 79.3 mm
- net Net-(IC1-Pad2): track 0.00 -> 75.7 mm
- net Net-(IC5-Pad6): track 0.00 -> 72.5 mm, vias 0 -> 2
- net Net-(R2-Pad3): track 64.4 -> 0.00 mm
- net Net-(IC1-Pad4): track 0.00 -> 51.4 mm, vias 0 -> 2
- net /A0: track 91.0 -> 129.4 mm
- net /A2: track 0.00 -> 33.6 mm, vias 0 -> 1
- net /A3: track 0.00 -> 33.3 mm, vias 0 -> 1
- net +5V: track 115.5 -> 148.3 mm, vias 2 -> 0
- net Net-(IC3-Pad7): track 26.5 -> 0.00 mm
- net Net-(IC3-Pad5): track 25.4 -> 0.00 mm
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- added copper zone on F.Cu, net +3.3V
- added copper zone on F.Cu, net +5V
- added copper zone on F.Cu, net GND
- added copper zone on B.Cu, net Net-(J3-Pad1)
- added copper zone on F.Cu, net Net-(J3-Pad1)
- added copper zone on B.Cu, net Net-(J3-Pad2)
- added copper zone on F.Cu, net Net-(J3-Pad2)
- added copper zone on B.Cu, net Net-(J4-Pad1)
- added copper zone on F.Cu, net Net-(J4-Pad1)
- added copper zone on B.Cu, net Net-(J4-Pad2)
- added copper zone on F.Cu, net Net-(J4-Pad2)
Other:
- board text added: "(10) 1"
- board text added: "(A2) 2"
- board text added: "(A3) 3"
- board text added: "1(A0)"
- board text added: "2(A1)"
- board text added: "3(9)"
- board text added: "RESET"
- board text added: "START"
- board text added: "Yet Another Reflow Toaster Controller"
- board text added: "https://github.com/takagiwa/mt_reflowcnt"

Commit message: レベルシフタの方向を修正
Parts:
- added TP1: TestPoint, TestPoint:TestPoint_Pad_D2.0mm, F.Cu at (145.0, 81.2)
- added TP2: TestPoint, TestPoint:TestPoint_Pad_D2.0mm, F.Cu at (199.6, 111.6)
- added TP3: TestPoint, TestPoint:TestPoint_Pad_D2.0mm, F.Cu at (183.9, 111.4)
- moved R2 0.54 mm to (254.0, 93.0)
- moved R5 0.54 mm to (254.0, 103.1)
- moved R4 0.52 mm to (254.0, 98.0)
- moved D2 0.51 mm to (254.0, 100.6)
- moved D3 0.51 mm to (254.0, 105.7)
- moved D1 0.49 mm to (254.0, 95.5)
- moved IC2 0.25 mm to (166.6, 91.1)
Connections:
- IC2 pad 2: Net-(IC2-Pad2) -> GND
- IC2 pad 3: GND -> Net-(IC3-Pad7)
- IC3 pad 7: Net-(IC2-Pad2) -> Net-(IC3-Pad7)
- IC4 pad 7: Net-(IC2-Pad2) -> Net-(IC3-Pad7)
- IC5 pad 7: Net-(IC2-Pad2) -> Net-(IC3-Pad7)
- R18 pad 2: Net-(IC2-Pad2) -> Net-(IC3-Pad7)
Routing:
- net Net-(IC3-Pad7): track 0.00 -> 81.3 mm
- net Net-(IC2-Pad2): track 79.3 -> 0.00 mm
- net GND: track 652.3 -> 660.2 mm, vias 49 -> 48
- net Net-(IC1-Pad3): track 29.3 -> 35.2 mm
- net Net-(IC1-Pad2): track 75.7 -> 77.1 mm
