File: kicad/mt_reflowcnt/mt_reflowcnt.kicad_sch (KiCad schematic)
At the start: 44 parts, among them IC1 TXB0101DBVR, IC2 TXB0101DBVR, IC3 MAX31855KASA+, IC4 NUP2105LT1G, IC5 TXB0101DBVR, J1 Conn_01x04, J2 PCC-SMP, P1 Power, P2 Analog, P3 Digital, P4 Digital, P5 CONN_01X01, P6 CONN_01X01, P7 CONN_01X01, P8 CONN_01X01, U1 SC2004CS_B

Commit message: first refined version. add more thermocouple and add one more relay control.
Parts:
- removed C1, C2, C3, C4, C6, C7, C8: 0.1u, Capacitor_SMD:C_0805_2012Metric_Pad1.18x1.45mm_HandSolder, symbol Device:C_Small
- removed C5: 0.01u, Capacitor_SMD:C_0805_2012Metric_Pad1.18x1.45mm_HandSolder, symbol Device:C_Small
- removed IC1, IC2, IC5: TXB0101DBVR, LibraryLoader:SOT95P280X145-6N, symbol LibraryLoader:TXB0101DBVR
- removed IC3: MAX31855KASA+, LibraryLoader:SOIC127P600X175-8N, symbol LibraryLoader:MAX31855KASA+
- removed IC4: NUP2105LT1G, LibraryLoader:SOT96P237X111-3N, symbol LibraryLoader:NUP2105LT1G
- removed J1: Conn_01x04, Connector_PinHeader_2.54mm:PinHeader_1x04_P2.54mm_Vertical, symbol Connector_Generic:Conn_01x04
- removed J2: PCC-SMP, mt_reflowcnt:PCC-SMP, symbol mt_reflowcnt:PCC-SMP
- removed L1, L2: 470ohm, Inductor_SMD:L_0603_1608Metric_Pad1.05x0.95mm_HandSolder, symbol Device:L_Small
- added D3: LED_Small, LED_SMD:LED_0805_2012Metric_Pad1.15x1.40mm_HandSolder, symbol Device:LED_Small
- added J1: Conn_01x06, Connector_PinHeader_2.54mm:PinHeader_1x06_P2.54mm_Vertical, symbol Connector_Generic:Conn_01x06
- added J5, J6, J7, J8: Conn_01x01, Connector_PinSocket_2.54mm:PinSocket_1x01_P2.54mm_Vertical, symbol Connector_Generic:Conn_01x01
- added R5: 220, Resistor_SMD:R_0805_2012Metric_Pad1.20x1.40mm_HandSolder, symbol Device:R_Small
- renumbered H2 to H1, H1 to H2, R9 to R10, R10 to R11, R11 to R12, R12 to R13, R3 to R2, R2 to R3, R5 to R6, R6 to R7, R7 to R8, R8 to R9
Connections:
- net 9(**): now also J1.5 (Pin_5), R5.1
- net A0: now also J1.1 (Pin_1)
- net A1: now also J1.3 (Pin_3)
- net GND: now also D3.1 (K), J1.2 (Pin_2), J1.4 (Pin_4), J1.6 (Pin_6), J5.1 (Pin_1), J6.1 (Pin_1), J7.1 (Pin_1), J8.1 (Pin_1)
- net +3V3 renamed +3.3V
- new net: D3.2 (A), R5.2
- no-connect marks 18 -> 15
Other:
- added sheet thermo.kicad_sch (untitled.kicad_sch)
- note removed: "1.5mA"
- moved on the sheet: D1, D2, R2, R4
