File: kicad/mt_reflowcnt/untitled.kicad_sch (KiCad schematic)
At the start: 32 parts, among them IC1 TXB0104D, IC2 TXB0101DBVR, IC3 MAX31855KASA+, IC4 MAX31855KASA+, IC5 MAX31855KASA+, IC6 NUP2105LT1G, IC7 NUP2105LT1G, IC8 NUP2105LT1G, J2 PCC-SMP, J3 PCC-SMP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

Commit message: レベルシフタの方向を修正
Parts:
- added TP1, TP2, TP3: TestPoint, TestPoint:TestPoint_Pad_D2.0mm, symbol Connector:TestPoint
Connections:
- net GND: now also IC2.2 (GND); no longer IC2.3 (A)
- net MISO: now also TP1.1
- net at IC3.7 (SO), IC4.7 (SO), IC5.7 (SO)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: now also IC2.3 (A); no longer IC2.2 (GND)
- net at IC1.2 (A1), IC3.5 (SCK), IC4.5 (SCK)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: now also TP2.1
- net at IC1.3 (A2), IC3.6 (~{CS}): now also TP3.1
